File: daedalus.kicad_sch (KiCad schematic)
At the start: 1 part

Commit message: Daedalus Rev A PoC
Parts:
- removed U?: RP2040, rp2040:RP2040, symbol rpi-silicon:RP2040
- added C19: 10nF, Capacitor_SMD:C_0402_1005Metric, symbol Device:C
- added C20, C21: 100nF, Capacitor_SMD:C_0402_1005Metric, symbol Device:C
- added C22: 2.2nF, Capacitor_SMD:C_0402_1005Metric, symbol Device:C
- added J1: PWR, Connector_AMASS:AMASS_XT30PW-M_1x02_P2.50mm_Horizontal, symbol Connector_Generic:Conn_01x02
- added J2: Host, raspberrypi:Raspberry_Pi_HAT_2_3_4, symbol Connector:Raspberry_Pi_4
- added J3: IO Port, Connector_PinHeader_2.54mm:PinHeader_2x08_P2.54mm_Vertical, symbol Connector_Generic:Conn_02x08_Top_Bottom
- added J4: MCU_I2C, Connector_PinHeader_2.54mm:PinHeader_1x04_P2.54mm_Vertical, symbol Connector_Generic:Conn_01x04
- added J5: SWD, Connector_PinHeader_2.54mm:PinHeader_1x04_P2.54mm_Vertical, symbol Connector_Generic:Conn_01x04
- added U3: MPU-6050, Sensor_Motion:InvenSense_QFN-24_4x4mm_P0.5mm, symbol Sensor_Motion:MPU-6050
Connections:
- new net: C21.1, U3.10 (REGOUT)
- new net: J2.19 (MOSI_SPI0/GPIO10), J3.15 (Pin_15)
- new net: J2.21 (MISO_SPI0/GPIO09), J3.14 (Pin_14)
- new net: J2.23 (SCLK_SPI0/GPIO11), J3.16 (Pin_16)
- new net: J2.24 (~{CE0}_SPI0/GPIO08), J3.13 (Pin_13)
- new net: J2.26 (~{CE1}_SPI0/GPIO07), J3.12 (Pin_12)
- new net: J2.29 (GPCLK1/GPIO05), J3.10 (Pin_10)
- new net: J2.31 (GPCLK2/GPIO06), J3.11 (Pin_11)
- new net: J2.7 (GPCLK0/GPIO04), J3.9 (Pin_9)
- new net: C22.1, U3.20 (CPOUT)
- new net +3V3: C19.1, C20.1, J2.1 (3V3), J4.1 (Pin_1), J5.1 (Pin_1), U3.13 (VDD), U3.8 (VLOGIC)
- new net +5V: J2.2 (5V)
- new net GND: C19.2, C20.2, C21.2, C22.2, J2.14 (GND), J2.20 (GND), J2.25 (GND), J2.30 (GND), J2.34 (GND), J2.39 (GND), J2.6 (GND), J2.9 (GND), J4.4 (Pin_4), J5.4 (Pin_4), U3.11 (FSYNC), U3.18 (GND), U3.9 (AD0)
- new net MCU/cs: J2.12 (GPIO18/SPI1_~{CE0}/PCM_CLK/PWM0)
- new net MCU/enable: J2.33 (GPIO13/PWM1)
- new net MCU/gpio0: J3.1 (Pin_1)
- new net MCU/gpio1: J3.2 (Pin_2)
- new net MCU/gpio2: J3.3 (Pin_3)
- new net MCU/gpio3: J3.4 (Pin_4)
- new net MCU/gpio4: J3.5 (Pin_5)
- new net MCU/gpio5: J3.6 (Pin_6)
- new net MCU/gpio6: J3.7 (Pin_7)
- new net MCU/gpio7: J3.8 (Pin_8)
- new net MCU/miso: J2.35 (GPIO19/SPI1_MISO/PCM_FS)
- new net MCU/mosi: J2.38 (GPIO20/SPI1_MOSI/PCM_DIN/PWM1)
- new net MCU/sck: J2.40 (GPIO21/SPI1_SCLK/PCM_DOUT)
- new net MCU/swclk: J2.37 (GPIO26/SDIO_DAT2), J5.2 (Pin_2)
- new net MCU/swdio: J2.22 (GPIO25/SDIO_DAT1), J5.3 (Pin_3)
- new net MCU/uart_rx: J2.8 (GPIO14/UART_TXD)
- new net MCU/uart_tx: J2.10 (GPIO15/UART_RXD)
- new net power_supply/pwr_gnd: J1.1 (Pin_1)
- new net power_supply/pwr_vcc: J1.2 (Pin_2)
- new net scl: J4.3 (Pin_3), U3.23 (SCL)
- new net sda: J4.2 (Pin_2), U3.24 (SDA)
- no-connect marks 0 -> 6
Other:
- added sheet MCU (mcu.kicad_sch)
- added sheet power_supply (power_supply.kicad_sch)
- note added: "TODO: I2C EEPROM"
- title: (none) -> Daedalus

Commit message: added missing lcsc part number
Other:
- note added: "I2C Address: $68"
Changed lines of the file:
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@@
+		)
+	)
+	(text "I2C Address: $68"
+		(exclude_from_sim no)
+		(at 37.084 186.182 0)
+		(effects
+			(font
+				(size 1.27 1.27)
+			)
 		)
 	)

Commit message: fix raspberry pi hat pinout
Connections:
- net +3V3: now also J2.17 (3V3)
- net +5V: now also J2.4 (5V)

Commit message: Switch to vertical xt30 connector
Parts:
- J1: footprint Connector_AMASS:AMASS_XT30PW-M_1x02_P2.50mm_Horizontal -> Connector_AMASS:AMASS_XT30UPB-M_1x02_P5.0mm_Vertical
Changed lines of the file:
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@@
 			)
 		)
-		(property "Footprint" "Connector_AMASS:AMASS_XT30PW-M_1x02_P2.50mm_Horizontal"
+		(property "Footprint" "Connector_AMASS:AMASS_XT30UPB-M_1x02_P5.0mm_Vertical"
 			(at 19.05 31.75 0)
 			(effects
