File: daedalus.kicad_sch (KiCad schematic)
At the start: 10 parts, among them J1 PWR, J2 Host, J3 IO Port, J4 MCU_I2C, J5 SWD, U3 MPU-6050

Commit message: Rev C
Parts:
- removed J1: PWR, Connector_AMASS:AMASS_XT30UPB-M_1x02_P5.0mm_Vertical, symbol Connector_Generic:Conn_01x02
- added C8: 1uF, Capacitor_SMD:C_0402_1005Metric, symbol Device:C
- added D3: 3V3, LED_SMD:LED_0603_1608Metric, symbol Device:LED
- added D4: 5V, LED_SMD:LED_0603_1608Metric, symbol Device:LED
- added J6: uart0, Connector_PinHeader_2.54mm:PinHeader_1x04_P2.54mm_Vertical, symbol Connector_Generic:Conn_01x04
- added R3, R8: 10k, Resistor_SMD:R_0402_1005Metric, symbol Device:R
- added R6, R7: 1k, Resistor_SMD:R_0402_1005Metric, symbol Device:R
- added SW2: SHT, tactile_switches:TS-1088-AR02016, symbol Switch:SW_Push
- added TP1: TP_5V, TestPoint:TestPoint_Pad_2.0x2.0mm, symbol Connector:TestPoint
- added TP2: TP_3V3, TestPoint:TestPoint_Pad_2.0x2.0mm, symbol Connector:TestPoint
- added TP3: TP_GND, TestPoint:TestPoint_Pad_2.0x2.0mm, symbol Connector:TestPoint
- added U7: AP2112K-3.3, Package_TO_SOT_SMD:SOT-23-5, symbol Regulator_Linear:AP2112K-3.3
Connections:
- net +3V3: now also C8.1, D3.2 (A), J6.1 (Pin_1), R8.1, TP2.1, U7.5 (VOUT)
- net +5V: now also D4.2 (A), R3.1, TP1.1, U7.1 (VIN)
- net GND: now also C8.2, J6.4 (Pin_4), R6.1, R7.1, SW2.1, TP3.1, U7.2 (GND)
- net MCU/uart_rx: now also J6.2 (Pin_2)
- net MCU/uart_tx: now also J6.3 (Pin_3)
- net at J2.11 (GPIO17/SPI1_~{CE1}): now also R8.2, SW2.2
- new net: D3.1 (K), R7.2
- new net: R3.2, U7.3 (EN)
- new net: D4.1 (K), R6.2
Other:
- removed sheet power_supply
- note added: "3.3V, 600mA"
- note added: "5V supplied by the Raspberry Pi"
- note added: "5V, 6A Max"
- note added: "Shutdown"
- note removed: "TODO: I2C EEPROM"
- title: Daedalus -> Daedalus Robotics Controller
- moved on the sheet: C19, C20, C21, C22, J2, J3, J4, J5, U3
