File: mcu.kicad_sch (KiCad schematic)
At the start: 25 parts, among them SW1 RST, U4 W25Q128JVS, U5 MCU, Y1 12MHz

Commit message: added missing lcsc part number
Parts:
- Y1: LCSC (none) -> C20625731
Changed lines of the file:
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@@
+			)
+		)
+		(property "LCSC" "C20625731"
+			(at 68.58 128.27 90)
+			(effects
+				(font
+					(size 1.27 1.27)
+				)
+				(hide yes)
 			)
 		)
