File: mcu.kicad_sch (KiCad schematic)
At the start: 25 parts, among them SW1 RST, U4 W25Q128JVS, U5 MCU, Y1 12MHz

Commit message: Rev C
Other:
- title: (none) -> Daedalus Robotics Controller
Changed lines of the file:
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@@
 	(paper "A4")
 	(title_block
-		(rev "B")
+		(title "Daedalus Robotics Controller")
+		(date "2026-07-01")
+		(rev "C")
 	)
 	(text "Place close to Pins 44 and 45"
