File: daedalus.kicad_pcb (KiCad board)
At the start: 4 copper layers, 65 x 56.5 mm, 57 parts, among them J1 PWR, J2 Host, J3 IO Port, J4 MCU_I2C, J5 SWD, U3 MPU-6050, U4 W25Q128JVS, U5 MCU, U6 TPS56637, U7 AP2112K-3.3, Y1 12MHz

Commit message: Rev C
Parts:
- removed C6: 4.7uF, Capacitor_SMD:C_0805_2012Metric
- removed C7, Cboot1: 100nF, Capacitor_SMD:C_0402_1005Metric
- removed Cff1: 100pF, Capacitor_SMD:C_0402_1005Metric
- removed Cout1: 47uF, Capacitor_SMD:C_0805_2012Metric
- removed J1: PWR, Connector_AMASS:AMASS_XT30UPB-M_1x02_P5.0mm_Vertical
- removed L2: 3.3uH, inductors:IHLP2525CZER3R3M01
- removed Rfbb1: 10k, Resistor_SMD:R_0402_1005Metric
- removed Rfbt1: 73.2k, Resistor_SMD:R_0402_1005Metric
- removed Rff1: 20k, Resistor_SMD:R_0402_1005Metric
- removed Rpg1: 100k, Resistor_SMD:R_0402_1005Metric
- removed U6: TPS56637, package_qfn_ext:VQFN-10-3x3mm
- added J6: uart0, Connector_PinHeader_2.54mm:PinHeader_1x04_P2.54mm_Vertical, F.Cu at (122.5, 76.9)
- added SW2: SHT, tactile_switches:TS-1088-AR02016, F.Cu at (123.0, 96.5)
- moved C8 19.0 mm to (128.9, 70.9)
- moved R3 19.0 mm to (123.0, 70.4)
- moved U7 19.0 mm to (126.0, 71.0)
- moved D1 4.89 mm to (122.4, 87.5)
- moved R4 4.89 mm to (125.5, 87.5)
- moved R2 4.89 mm to (126.7, 92.5)
- moved D2 4.89 mm to (122.4, 89.3)
- moved R5 4.89 mm to (125.5, 89.4)
- moved SW1 4.89 mm to (122.9, 92.4)
- renumbered RST to SW1
Connections:
- J2 pad 11: unconnected-(J2-GPIO17/SPI1_~{CE1}-Pad11) -> Net-(J2-GPIO17/SPI1_~{CE1})
Routing:
- net Net-(J2-GPIO17/SPI1_~{CE1}): track 0.00 -> 46.8 mm, vias 0 -> 2
- net +5V: track 50.2 -> 6.55 mm, vias 3 -> 2
- net /MCU/uart_rx: track 42.9 -> 83.3 mm, vias 2 -> 4
- net /MCU/uart_tx: track 41.7 -> 78.1 mm, vias 2 -> 6
- net /power_supply/pwr_vcc: track 13.5 -> 0.00 mm
- net Net-(U6-FB): track 9.25 -> 0.00 mm
- net GND: track 64.1 -> 56.7 mm, vias 19 -> 16
- net Net-(U6-PG): track 7.36 -> 0.00 mm
- net Net-(D2-A): track 108.5 -> 114.6 mm
- net Net-(U6-SW): track 6.12 -> 0.00 mm
- net +3V3: track 76.2 -> 82.2 mm, vias 12 -> 11
- net Net-(D1-A): track 117.5 -> 123.1 mm
- net /MCU/run: track 135.7 -> 140.8 mm
- net Net-(J2-GPCLK0/GPIO04): track 51.4 -> 52.9 mm, vias 0 -> 1
- net Net-(U6-BOOT): track 1.44 -> 0.00 mm
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- removed copper zone on In1.Cu, net /power_supply/pwr_vcc
Other:
- board text added: "RX"
- board text added: "Shutdown"
- board text added: "TX"
