File: power_supply.kicad_sch (KiCad schematic)
At the start: 21 parts, among them U6 TPS56637, U7 AP2112K-3.3

Commit message: Rev C
Parts:
- removed C6: 4.7uF, Capacitor_SMD:C_0805_2012Metric, symbol Device:C
- removed C7, Cboot1: 100nF, Capacitor_SMD:C_0402_1005Metric, symbol Device:C
- removed C8: 1uF, Capacitor_SMD:C_0402_1005Metric, symbol Device:C
- removed Cff1: 100pF, Capacitor_SMD:C_0402_1005Metric, symbol Device:C
- removed Cout1: 47uF, Capacitor_SMD:C_0805_2012Metric, symbol Device:C
- removed D3: 3V3, LED_SMD:LED_0603_1608Metric, symbol Device:LED
- removed D4: 5V, LED_SMD:LED_0603_1608Metric, symbol Device:LED
- removed L2: 3.3uH, inductors:IHLP2525CZER3R3M01, symbol Device:L
- removed R3, Rfbb1: 10k, Resistor_SMD:R_0402_1005Metric, symbol Device:R
- removed R6, R7: 1k, Resistor_SMD:R_0402_1005Metric, symbol Device:R
- removed Rfbt1: 73.2k, Resistor_SMD:R_0402_1005Metric, symbol Device:R
- removed Rff1: 20k, Resistor_SMD:R_0402_1005Metric, symbol Device:R
- removed Rpg1: 100k, Resistor_SMD:R_0402_1005Metric, symbol Device:R
- removed TP1: TP_5V, TestPoint:TestPoint_Pad_2.0x2.0mm, symbol Connector:TestPoint
- removed TP2: TP_3V3, TestPoint:TestPoint_Pad_2.0x2.0mm, symbol Connector:TestPoint
- removed TP3: TP_GND, TestPoint:TestPoint_Pad_2.0x2.0mm, symbol Connector:TestPoint
- removed U6: TPS56637, package_qfn_ext:VQFN-10-3x3mm, symbol power_supply:TPS56637
- removed U7: AP2112K-3.3, Package_TO_SOT_SMD:SOT-23-5, symbol Regulator_Linear:AP2112K-3.3
Connections:
- no-connect marks 1 -> 0
Other:
- note removed: "3.3V, 600mA"
- note removed: "5V, 6A Max"
- note removed: "7V - 25V Input 2S - 6S LiPo"
- note removed: "Power Supply"
